Commit message: real2sim 추가

File: source/robot_lab/data/Robots/rnd/step/urdf/step.urdf (robot description, URDF)
Before this commit: robot step, 24 links, 23 joints
Links:
- link L_Arm_hand: mass 0.014931 -> 0.018532
- link L_Arm_lower: mass 0.11579 -> 0.11139
- link R_Arm_hand: mass 0.014931 -> 0.018532
- link R_Arm_lower: mass 0.11579 -> 0.11139
- link Upper_Body: mass 1.6979 -> 1.6853
Joints:
- joint L_Leg_ankle_pitch: limit lower=-0.41 upper=1.47 effort=5.4 velocity=4.18 -> lower=-3.14159265358979 upper=3.14159265358979 effort=8.4 velocity=4.71238898038469
- joint L_Leg_ankle_roll: limit lower=-1.57 upper=1.57 effort=5.4 velocity=4.18 -> lower=-3.14159265358979 upper=3.14159265358979 effort=8.4 velocity=4.71238898038469
- joint L_Leg_hip_pitch: limit lower=-0.25 upper=1.90 effort=5.4 velocity=4.18 -> lower=-3.14159265358979 upper=3.14159265358979 effort=8.4 velocity=4.71238898038469; origin xyz=0.0308 -0.03589 -0.07773 rpy=3.1416 -1.5708 0 -> xyz=0.0308 -0.03589 -0.07773 rpy=0 -1.5708 -3.1416
- joint L_Leg_hip_roll: limit lower=-1.40 upper=1.40 effort=5.4 velocity=4.18 -> lower=-3.14159265358979 upper=3.14159265358979 effort=8.4 velocity=4.71238898038469; origin xyz=0.07904 -0.0005 0.030391 rpy=-1.5708 0 -1.5708 -> xyz=0.0790399999998856 -0.000500004039074131 0.0303914536643952 rpy=-1.57079632680575 0 -1.57079632676978
- joint L_Leg_hip_yaw: limit lower=-0.64 upper=0.64 effort=5.4 velocity=4.18 -> lower=-3.14159265358979 upper=3.14159265358979 effort=8.4 velocity=4.71238898038469
- joint L_Leg_knee: limit lower=-2.12 upper=1.13 effort=5.4 velocity=4.18 -> lower=-3.14159265358979 upper=3.14159265358979 effort=8.4 velocity=4.71238898038469
- joint Neck_yaw: origin xyz=0 -0.040141 0.11705 rpy=0 0 3.1416 -> xyz=0 -0.040141 0.14855 rpy=0 0 3.1416
- joint R_Leg_ankle_pitch: limit lower=-1.47 upper=0.41 effort=5.4 velocity=4.18 -> lower=-3.14159265358979 upper=3.14159265358979 effort=8.4 velocity=4.71238898038469
- joint R_Leg_ankle_roll: limit lower=-1.57 upper=1.57 effort=5.4 velocity=4.18 -> lower=-3.14159265358979 upper=3.14159265358979 effort=8.4 velocity=4.71238898038469; origin xyz=0.07773 -0.03589 -0.0308 rpy=3.1416 -1.5708 0 -> xyz=0.07773 -0.03589 -0.0308 rpy=0 -1.5708 3.1416
- joint R_Leg_hip_pitch: limit lower=-1.90 upper=0.25 effort=5.4 velocity=4.18 -> lower=-3.14159265358979 upper=3.14159265358979 effort=8.4 velocity=4.71238898038469
- joint R_Leg_hip_roll: limit lower=-1.40 upper=1.40 effort=5.4 velocity=4.18 -> lower=-3.14159265358979 upper=3.14159265358979 effort=8.4 velocity=4.71238898038469
- joint R_Leg_hip_yaw: limit lower=-0.64 upper=0.64 effort=5.4 velocity=4.18 -> lower=-3.14159265358979 upper=3.14159265358979 effort=8.4 velocity=4.71238898038469
- joint R_Leg_knee: limit lower=-1.13 upper=2.12 effort=5.4 velocity=4.18 -> lower=-3.14159265358979 upper=3.14159265358979 effort=8.4 velocity=4.71238898038469
