Commit message: real2sim and imu_2

File: source/robot_lab/data/Robots/rnd/STEP URDF IMU/urdf/STEP URDF IMU.urdf (robot description, URDF)
Before this commit: robot step, 25 links, 24 joints
Links:
- link L_Arm_hand: geometry collision mesh filename=package://STEP URDF IMU/meshes/L_Arm_hand.STL; visual mesh filename=package://STEP URDF IMU/meshes/L_Arm_hand.STL
- link L_Arm_lower: geometry collision mesh filename=package://STEP URDF IMU/meshes/L_Arm_lower.STL; visual mesh filename=package://STEP URDF IMU/meshes/L_Arm_lower.STL
- link L_Arm_shoulder: geometry collision mesh filename=package://STEP URDF IMU/meshes/L_Arm_shoulder.STL; visual mesh filename=package://STEP URDF IMU/meshes/L_Arm_shoulder.STL
- link L_Arm_upper: geometry collision mesh filename=package://STEP URDF IMU/meshes/L_Arm_upper.STL; visual mesh filename=package://STEP URDF IMU/meshes/L_Arm_upper.STL
- link L_Leg_ankle: geometry collision mesh filename=package://STEP URDF IMU/meshes/L_Leg_ankle.STL; visual mesh filename=package://STEP URDF IMU/meshes/L_Leg_ankle.STL
- link L_Leg_calf: geometry collision mesh filename=package://STEP URDF IMU/meshes/L_Leg_calf.STL; visual mesh filename=package://STEP URDF IMU/meshes/L_Leg_calf.STL
- link L_Leg_foot: geometry collision mesh filename=package://STEP URDF IMU/meshes/L_Leg_foot.STL; visual mesh filename=package://STEP URDF IMU/meshes/L_Leg_foot.STL
- link L_Leg_hip: geometry collision mesh filename=package://STEP URDF IMU/meshes/L_Leg_hip.STL; visual mesh filename=package://STEP URDF IMU/meshes/L_Leg_hip.STL
- link L_Leg_hip_double: geometry collision mesh filename=package://STEP URDF IMU/meshes/L_Leg_hip_double.STL; visual mesh filename=package://STEP URDF IMU/meshes/L_Leg_hip_double.STL
- link L_Leg_thighs: geometry collision mesh filename=package://STEP URDF IMU/meshes/L_Leg_thighs.STL; visual mesh filename=package://STEP URDF IMU/meshes/L_Leg_thighs.STL
- link Neck: geometry collision mesh filename=package://STEP URDF IMU/meshes/Neck.STL; visual mesh filename=package://STEP URDF IMU/meshes/Neck.STL
- link R_Arm_hand: geometry collision mesh filename=package://STEP URDF IMU/meshes/R_Arm_hand.STL; visual mesh filename=package://STEP URDF IMU/meshes/R_Arm_hand.STL
- link R_Arm_lower: geometry collision mesh filename=package://STEP URDF IMU/meshes/R_Arm_lower.STL; visual mesh filename=package://STEP URDF IMU/meshes/R_Arm_lower.STL
- link R_Arm_shoulder: geometry collision mesh filename=package://STEP URDF IMU/meshes/R_Arm_shoulder.STL; visual mesh filename=package://STEP URDF IMU/meshes/R_Arm_shoulder.STL
- link R_Arm_upper: geometry collision mesh filename=package://STEP URDF IMU/meshes/R_Arm_upper.STL; visual mesh filename=package://STEP URDF IMU/meshes/R_Arm_upper.STL
- link R_Leg_ankle: geometry collision mesh filename=package://STEP URDF IMU/meshes/R_Leg_ankle.STL; visual mesh filename=package://STEP URDF IMU/meshes/R_Leg_ankle.STL
- link R_Leg_calf: geometry collision mesh filename=package://STEP URDF IMU/meshes/R_Leg_calf.STL; visual mesh filename=package://STEP URDF IMU/meshes/R_Leg_calf.STL
- link R_Leg_foot: geometry collision mesh filename=package://STEP URDF IMU/meshes/R_Leg_foot.STL; visual mesh filename=package://STEP URDF IMU/meshes/R_Leg_foot.STL
- link R_Leg_hip: geometry collision mesh filename=package://STEP URDF IMU/meshes/R_Leg_hip.STL; visual mesh filename=package://STEP URDF IMU/meshes/R_Leg_hip.STL
- link R_Leg_hip_double: geometry collision mesh filename=package://STEP URDF IMU/meshes/R_Leg_hip_double.STL; visual mesh filename=package://STEP URDF IMU/meshes/R_Leg_hip_double.STL
- link R_Leg_thighs: geometry collision mesh filename=package://STEP URDF IMU/meshes/R_Leg_thighs.STL; visual mesh filename=package://STEP URDF IMU/meshes/R_Leg_thighs.STL
- link Upper_Body: geometry collision mesh filename=package://STEP URDF IMU/meshes/Upper_Body.STL; visual mesh filename=package://STEP URDF IMU/meshes/Upper_Body.STL
- link base_link: geometry collision mesh filename=package://STEP URDF IMU/meshes/base_link.STL; visual mesh filename=package://STEP URDF IMU/meshes/base_link.STL
- link head: geometry collision mesh filename=package://STEP URDF IMU/meshes/head.STL; visual mesh filename=package://STEP URDF IMU/meshes/head.STL
- link imu: geometry collision mesh filename=package://STEP URDF IMU/meshes/imu.STL; visual mesh filename=package://STEP URDF IMU/meshes/imu.STL
Joints:
- joint imu_body: origin xyz=6.5633E-05 0.013628 0.11395 rpy=0 0 3.141592653589793 -> xyz=6.5633E-05 0.013628 0.11395 rpy=0 0 3.1416
